File: power-toggle-on-hold-off/power-toggle-on-hold-off.sch (KiCad schematic (older format))
At the start: 13 parts, among them J1 VIN, SW1 POWER, U1 BSD235C

Commit message: Updated on-off schematics for verification, last one did not work :-)
Signed-off-by: Tomasz 'CeDeROM' CEDRO <tomek@cedro.info>
Parts:
- added C2, C4, C7: ???, Capacitor_SMD:C_0805_2012Metric_Pad1.15x1.40mm_HandSolder, symbol Device:C
- added C3: 100nF, Capacitor_SMD:C_0805_2012Metric_Pad1.15x1.40mm_HandSolder, symbol Device:C
- added C5: 1uF, Capacitor_SMD:C_0805_2012Metric_Pad1.15x1.40mm_HandSolder, symbol Device:C
- added C6: 10uF, Capacitor_SMD:C_0805_2012Metric_Pad1.15x1.40mm_HandSolder, symbol Device:C
- added D1: 1N4148, Diode_SMD:D_0805_2012Metric, symbol Device:D
- added R1: 10k, Resistor_SMD:R_0603_1608Metric_Pad1.05x0.95mm_HandSolder, symbol Device:R
- added R3: ???, Resistor_SMD:R_0603_1608Metric_Pad1.05x0.95mm_HandSolder, symbol Device:R
- added R6: 100K, Resistor_SMD:R_0603_1608Metric_Pad1.05x0.95mm_HandSolder, symbol Device:R
- added SW2: POWERONDEF, Jumper:SolderJumper-3_P1.3mm_Bridged12_RoundedPad1.0x1.5mm_NumberLabels, symbol Switch:SW_Push_SPDT
- added TP2: VCAP, TestPoint:TestPoint_Pad_D2.0mm, symbol Connector:TestPoint
- C1: value 10uF -> 1uF
- D2: renamed from D1; symbol CeDeROM_Device:LED -> Device:LED
- R2: value 1M -> ???
- R4: renamed from R1; value 10K -> 100k
- R5: renamed from R3; value 10K -> 300K
- SW1: footprint Button_Switch_SMD:SW_SPST_EVQP0 -> Button_Switch_SMD:SW_SPST_B3U-3000P
- TP3: renamed from TP2; value VCAP -> VGD
- TP4: renamed from TP3; value BUTTON -> PWRCTL
- renumbered R4 to R7, TP4 to TP5
Connections:
- net GND: now also SW1.1, SW2.3 (C); no longer C1.2
- net VCC: now also R2.1, R1.1, R3.1, SW2.1 (A)
- net at R5.2, U1.2 (GN): now also C5.1, C6.1, C7.1; no longer SW1.2, TP4.1
- net at R7.1, TP5.1, U1.3 (DP): now also C5.2, C6.2, C7.2, R6.2; no longer R5.1
- net at R4.2, U1.5 (GP), U1.6 (DN): now also C1.1, TP3.1, C2.1, C3.1, C4.1, R3.2; no longer R2.1
- new net: C1.2, C2.2, D1.1 (K), R1.2, R2.2, SW1.2, TP2.1
- new net: D1.2 (A), R5.1, R6.1, TP4.1
- new net: C3.2, C4.2, SW2.2 (B)
Other:
- note added: "NOTES:\n1. Push button short to Power-ON. Hold button to Power-OFF.\n2. SW1 selects default power-attach state as ON or OFF.\n3. Additional ??? places for R and C for experimental values.\n\nSOURCE: http://www.mosaic-industries.com/embedded-systems/microcontroller-projects/"
- note added: "OFF\nON"
- moved on the sheet: C1, D2, J1, R2, R4, R5, R7, SW1, TP1, TP3, TP4, TP5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
